File: neolexis/output/pcbs/left.kicad_pcb (KiCad board)
At the start: 2 copper layers, 151.4 x 119.5 mm, 77 parts

Commit message: feat: schematic first try
Parts:
- removed ? (x5): , HOLE_M2_TH
- moved T1 87.6 mm to (166.8, 144.4)
- moved D10 82.6 mm to (105.1, 133.4)
- moved D13 82.6 mm to (124.1, 169.4)
- moved D14 82.6 mm to (124.1, 150.4)
- moved D16 82.6 mm to (143.1, 167.4)
- moved D17 82.6 mm to (143.1, 148.4)
- moved D18 82.6 mm to (143.1, 129.4)
- moved D32 82.6 mm to (105.1, 145.4)
- moved D33 82.6 mm to (124.1, 132.4)
- moved D9 82.6 mm to (105.1, 171.4)
- moved D1 82.6 mm to (67.1, 156.4)
- moved D11 82.6 mm to (105.1, 114.4)
- moved D12 82.6 mm to (105.1, 95.4)
- moved D15 82.6 mm to (124.1, 112.4)
- moved D19 82.6 mm to (143.1, 110.4)
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Other:
- board size 151.4 x 119.5 mm -> 177 x 118 mm
- net class Default removed
