File: neolexis/pcb/neolexis.kicad_pcb (KiCad board)
At the start: 2 copper layers, 177 x 118 mm, 72 parts

Commit message: feat: add reference
Parts:
- added D0: D, Keebio-Parts:Diode-dual, F.Cu at (234.4, -111.4)
- added D1: D, Keebio-Parts:Diode-dual, F.Cu at (256.0, -111.4)
- added D10: D, Keebio-Parts:Diode-dual, F.Cu at (234.4, -92.4)
- added D11: D, Keebio-Parts:Diode-dual, F.Cu at (256.0, -92.4)
- added D12: D, Keebio-Parts:Diode-dual, F.Cu at (275.1, -96.8)
- added D13: D, Keebio-Parts:Diode-dual, F.Cu at (294.1, -99.4)
- added D14: D, Keebio-Parts:Diode-dual, F.Cu at (313.2, -96.8)
- added D15: D, Keebio-Parts:Diode-dual, F.Cu at (332.2, -94.9)
- added D16: D, Keebio-Parts:Diode-dual, F.Cu at (351.3, -79.7)
- added D2: D, Keebio-Parts:Diode-dual, F.Cu at (275.1, -115.9)
- added D20: D, Keebio-Parts:Diode-dual, F.Cu at (234.4, -73.3)
- added D21: D, Keebio-Parts:Diode-dual, F.Cu at (256.0, -73.3)
- added D22: D, Keebio-Parts:Diode-dual, F.Cu at (275.1, -77.8)
- added D23: D, Keebio-Parts:Diode-dual, F.Cu at (294.1, -80.3)
- added D24: D, Keebio-Parts:Diode-dual, F.Cu at (313.2, -77.8)
- added D25: D, Keebio-Parts:Diode-dual, F.Cu at (332.2, -75.9)
- added D26: D, Keebio-Parts:Diode-dual, F.Cu at (350.6, -51.7)
- added D3: D, Keebio-Parts:Diode-dual, F.Cu at (294.1, -118.4)
- added D30: D, Keebio-Parts:Diode-dual, F.Cu at (234.4, -54.3)
- added D31: D, Keebio-Parts:Diode-dual, F.Cu at (256.0, -54.3)
- added D32: D, Keebio-Parts:Diode-dual, F.Cu at (275.1, -58.7)
- added D33: D, Keebio-Parts:Diode-dual, F.Cu at (294.1, -61.3)
- added D34: D, Keebio-Parts:Diode-dual, F.Cu at (313.2, -58.7)
- added D35: D, Keebio-Parts:Diode-dual, F.Cu at (332.2, -56.8)
- added D36: D, Keebio-Parts:Diode-dual, F.Cu at (367.2, -42.2)
- added D4: D, Keebio-Parts:Diode-dual, F.Cu at (313.2, -115.9)
- added D40: D, Keebio-Parts:Diode-dual, F.Cu at (246.5, -43.5)
- added D41: D, Keebio-Parts:Diode-dual, F.Cu at (265.6, -45.4)
- added D42: D, Keebio-Parts:Diode-dual, F.Cu at (284.6, -47.9)
- added D43: D, Keebio-Parts:Diode-dual, F.Cu at (303.7, -50.5)
- added D44: D, Keebio-Parts:Diode-dual, F.Cu at (331.0, -41.8)
- added D45: D, Keebio-Parts:Diode-dual, F.Cu at (338.3, -30.4)
- added D46: D, Keebio-Parts:Diode-dual, F.Cu at (355.1, -20.7)
- added D5: D, Keebio-Parts:Diode-dual, F.Cu at (332.2, -114.0)
- added D6: D, Keebio-Parts:Diode-dual, F.Cu at (351.3, -104.4)
- added G***: LOGO, myparts:redox-logo, F.Cu at (245.2, -83.5)
- added G***: LOGO, myparts:qmk-badge, F.Cu at (322.6, -134.4)
- added G***: LOGO, myparts:qmk-badge, B.Cu at (323.6, -134.4)
- added G***: LOGO, myparts:redox-logo, B.Cu at (245.2, -84.1)
- added HOLE_M3: VAL**, keyboard_parts:HOLE_M3, F.Cu at (339.2, -134.3)
- added HOLE_M3: VAL**, keyboard_parts:HOLE_M3, F.Cu at (228.7, -132.4)
- added HOLE_M3: VAL**, keyboard_parts:HOLE_M3, F.Cu at (356.4, -42.1)
- added HOLE_M3: VAL**, keyboard_parts:HOLE_M3, F.Cu at (245.9, -57.4)
- added K0: KEYSW, myparts:Mx_Alps_125-dualside, F.Cu at (234.4, -119.7)
- added K1: KEYSW, canadian_footprints:Mx_Alps_100-dualside, F.Cu at (256.0, -119.7)
- added K10: KEYSW, myparts:Mx_Alps_125-dualside, F.Cu at (234.4, -100.6)
- added K11: KEYSW, canadian_footprints:Mx_Alps_100-dualside, F.Cu at (256.0, -100.6)
- added K12: KEYSW, canadian_footprints:Mx_Alps_100-dualside, F.Cu at (275.1, -105.1)
- added K13: KEYSW, canadian_footprints:Mx_Alps_100-dualside, F.Cu at (294.1, -107.6)
- added K14: KEYSW, canadian_footprints:Mx_Alps_100-dualside, F.Cu at (313.2, -105.1)
- added K15: KEYSW, canadian_footprints:Mx_Alps_100-dualside, F.Cu at (332.2, -103.2)
- added K16: KEYSW, canadian_footprints:Mx_Alps_150-dualsided, F.Cu at (351.3, -88.6)
- added K2: KEYSW, canadian_footprints:Mx_Alps_100-dualside, F.Cu at (275.1, -124.1)
- added K20: KEYSW, myparts:Mx_Alps_125-dualside, F.Cu at (234.4, -81.6)
- added K21: KEYSW, canadian_footprints:Mx_Alps_100-dualside, F.Cu at (256.0, -81.6)
- added K22: KEYSW, canadian_footprints:Mx_Alps_100-dualside, F.Cu at (275.1, -86.0)
- added K23: KEYSW, canadian_footprints:Mx_Alps_100-dualside, F.Cu at (294.1, -88.6)
- added K24: KEYSW, canadian_footprints:Mx_Alps_100-dualside, F.Cu at (313.2, -86.0)
- added K25: KEYSW, canadian_footprints:Mx_Alps_100-dualside, F.Cu at (332.2, -84.1)
- added K26: KEYSW, canadian_footprints:Mx_Alps_100-dualside, F.Cu at (355.1, -58.7)
- added K3: KEYSW, canadian_footprints:Mx_Alps_100-dualside, F.Cu at (294.1, -126.7)
- added K30: KEYSW, myparts:Mx_Alps_125-dualside, F.Cu at (234.4, -62.5)
- added K31: KEYSW, canadian_footprints:Mx_Alps_100-dualside, F.Cu at (256.0, -62.5)
- added K32: KEYSW, canadian_footprints:Mx_Alps_100-dualside, F.Cu at (275.1, -67.0)
- added K33: KEYSW, canadian_footprints:Mx_Alps_100-dualside, F.Cu at (294.1, -69.5)
- added K34: KEYSW, canadian_footprints:Mx_Alps_100-dualside, F.Cu at (313.2, -67.0)
- added K35: KEYSW, canadian_footprints:Mx_Alps_100-dualside, F.Cu at (332.2, -65.1)
- added K36: KEYSW, canadian_footprints:Mx_Alps_100-dualside, F.Cu at (371.6, -49.2)
- added K4: KEYSW, canadian_footprints:Mx_Alps_100-dualside, F.Cu at (313.2, -124.1)
- added K40: KEYSW, canadian_footprints:Mx_Alps_100-dualside, F.Cu at (237.0, -43.5)
- added K41: KEYSW, canadian_footprints:Mx_Alps_100-dualside, F.Cu at (256.0, -43.5)
- added K42: KEYSW, canadian_footprints:Mx_Alps_100-dualside, F.Cu at (275.1, -47.9)
- added K43: KEYSW, canadian_footprints:Mx_Alps_100-dualside, F.Cu at (294.1, -50.5)
- added K44: KEYSW, myparts:Mx_Alps_125-dualside, F.Cu at (319.5, -44.7)
- added K45: KEYSW, canadian_footprints:Mx_Alps_150-dualsided, F.Cu at (343.0, -37.8)
- added K46: KEYSW, canadian_footprints:Mx_Alps_150-dualsided, F.Cu at (359.5, -28.2)
- added K5: KEYSW, canadian_footprints:Mx_Alps_100-dualside, F.Cu at (332.2, -122.2)
- added K6: KEYSW, canadian_footprints:Mx_Alps_100-dualside, F.Cu at (351.3, -112.7)
- added R1: 4.7k, Keebio-Parts:Resistor-Compact, F.Cu at (343.7, -126.9)
- added R2: 4.7k, Keebio-Parts:Resistor-Compact, F.Cu at (357.9, -126.9)
- added REF***: OSHW-Logo2_14.6x12mm_SilkScreen, Symbols:OSHW-Symbol_8.9x8mm_SilkScreen, F.Cu at (248.4, -131.7)
- added REF***: OSHW-Logo2_14.6x12mm_SilkScreen, Symbols:OSHW-Symbol_8.9x8mm_SilkScreen, B.Cu at (248.4, -131.7)
- added RGB_STRIP1: Conn_01x03, Pin_Headers:Pin_Header_Straight_1x03_Pitch2.54mm, F.Cu at (341.9, -84.7)
- added RST_SW1: SW_PUSH, Buttons_Switches_ThroughHole:SW_PUSH_6mm_h4.3mm, F.Cu at (257.8, -135.0)
- added TRRS1: Audio-Jack-4, Keebio-Parts:TRRS-PJ-320A-dual, F.Cu at (350.8, -135.5)
- added U1: ProMicro, Keebio-Parts:ArduinoProMicro, F.Cu at (294.1, -120.3)
Routing:
- net row3: track 0.00 -> 207.9 mm, vias 0 -> 1
- net row4: track 0.00 -> 189.3 mm
- net row2: track 0.00 -> 188.9 mm, vias 0 -> 1
- net col6: track 0.00 -> 184.3 mm
- net row1: track 0.00 -> 169.3 mm, vias 0 -> 1
- net col0: track 0.00 -> 167.6 mm
- net col5: track 0.00 -> 146.1 mm
- net col1: track 0.00 -> 144.0 mm
- net row0: track 0.00 -> 135.3 mm
- net col2: track 0.00 -> 119.8 mm
- net rgb_data: track 0.00 -> 103.7 mm, vias 0 -> 2
- net col4: track 0.00 -> 103.1 mm
- net VCC: track 0.00 -> 103.1 mm
- net col3: track 0.00 -> 97.8 mm
- net SCL: track 0.00 -> 80.1 mm, vias 0 -> 2
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- added copper zone on B.Cu, net (none)
- added copper zone on F.Cu, net (none)
- added copper zone on B.Cu, net GND
- added copper zone on F.Cu, net GND
Other:
- board size 177 x 118 mm -> 338.7 x 279.6 mm
- board text added: "LEFT"
- board text added: "RIGHT"
- board text added: "designed by Mattia Dal Ben (https://github.com/mattdibi)"
- board text added: "rev 1.0"

Commit message: feat: cluster outline
Parts:
- removed D36, D46: D, Keebio-Parts:Diode-dual
- removed G*** (x2): LOGO, myparts:redox-logo
- removed G*** (x2): LOGO, myparts:qmk-badge
- removed K16: KEYSW, canadian_footprints:Mx_Alps_150-dualsided
- removed REF*** (x2): OSHW-Logo2_14.6x12mm_SilkScreen, Symbols:OSHW-Symbol_8.9x8mm_SilkScreen
- added HOLE_M3: VAL**, keyboard_parts:HOLE_M3, F.Cu at (360.8, -108.5)
- added K46: KEYSW, PCM_Switch_Keyboard_Hotswap_Kailh:SW_Hotswap_Kailh_Choc_V1V2_1.25u_90deg, F.Cu at (398.5, -90.7)
- added REF**: SW_Hotswap_Kailh_Choc_V1V2_1.50u_90deg, PCM_Switch_Keyboard_Hotswap_Kailh:SW_Hotswap_Kailh_Choc_V1V2_1.50u_90deg, F.Cu at (338.0, -85.0)
- added REF**: SW_Hotswap_Kailh_Choc_V1V2_1.50u, PCM_Switch_Keyboard_Hotswap_Kailh:SW_Hotswap_Kailh_Choc_V1V2_1.50u, F.Cu at (377.5, -112.2)
- added REF**: Harting_har-flexicon_14110213001xxx_1x02-MP_P2.54mm_Vertical, Connector_Harting:Harting_har-flexicon_14110213001xxx_1x02-MP_P2.54mm_Vertical, F.Cu at (355.2, -107.8)
- added REF**: Harting_har-flexicon_14110213001xxx_1x02-MP_P2.54mm_Vertical, Connector_Harting:Harting_har-flexicon_14110213001xxx_1x02-MP_P2.54mm_Vertical, F.Cu at (341.6, -45.7)
- K0, K10, K20, K30: footprint myparts:Mx_Alps_125-dualside -> PCM_Switch_Keyboard_Hotswap_Kailh:SW_Hotswap_Kailh_Choc_V1V2_1.25u
- K1, K11, K12, K13, K14, K15, K2, K21, K22, K23, K24, K25, K26, K3, K31, K32, K33, K34, K35, K4, K40, K41, K42, K43, K5, K6: footprint canadian_footprints:Mx_Alps_100-dualside -> PCM_Switch_Keyboard_Hotswap_Kailh:SW_Hotswap_Kailh_Choc_V1V2_1.00u
- K36: footprint canadian_footprints:Mx_Alps_100-dualside -> PCM_Switch_Keyboard_Hotswap_Kailh:SW_Hotswap_Kailh_Choc_V1V2_1.25u_90deg
- K44: footprint myparts:Mx_Alps_125-dualside -> PCM_Switch_Keyboard_Hotswap_Kailh:SW_Hotswap_Kailh_Choc_V1V2_1.00u
- K45: footprint canadian_footprints:Mx_Alps_150-dualsided -> PCM_Switch_Keyboard_Hotswap_Kailh:SW_Hotswap_Kailh_Choc_V1V2_1.00u
- K46: footprint canadian_footprints:Mx_Alps_150-dualsided -> PCM_Switch_Keyboard_Hotswap_Kailh:SW_Hotswap_Kailh_Choc_V1V2_1.25u_90deg
- moved B1 252.2 mm to (118.1, -174.8)
- moved D1 252.2 mm to (19.3, -144.8)
- moved D10 252.2 mm to (57.3, -167.8)
- moved D11 252.2 mm to (57.3, -186.8)
- moved D12 252.2 mm to (57.3, -205.8)
- moved D13 252.2 mm to (76.3, -131.8)
- moved D14 252.2 mm to (76.3, -150.8)
- moved D15 252.2 mm to (76.3, -188.8)
- moved D16 252.2 mm to (95.3, -133.8)
- moved D17 252.2 mm to (95.3, -152.8)
- moved D18 252.2 mm to (95.3, -171.8)
- moved D19 252.2 mm to (95.3, -190.8)
- moved D2 252.2 mm to (19.3, -163.8)
- moved D20 252.2 mm to (95.3, -209.8)
- moved D21 252.2 mm to (114.3, -185.8)
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Routing:
- net SDA: track 71.4 -> 184.6 mm
- net col5: track 146.1 -> 33.0 mm
- net row1: track 169.3 -> 192.9 mm
- net row3: track 207.9 -> 225.6 mm
- net row2: track 188.9 -> 200.8 mm
- net Net-(D31-Pad2): track 11.8 -> 0.00 mm
- net Net-(D21-Pad2): track 11.8 -> 0.00 mm
- net Net-(D11-Pad2): track 11.8 -> 0.00 mm
- net Net-(D25-Pad2): track 11.8 -> 0.00 mm
- net Net-(D1-Pad2): track 11.8 -> 0.00 mm
- net row0: track 135.3 -> 147.2 mm
- net Net-(D4-Pad2): track 11.8 -> 21.7 mm
- net col4: track 103.1 -> 93.2 mm
- net Net-(D46-Pad2): track 5.91 -> 0.00 mm
Other:
- board size 338.7 x 279.6 mm -> 408.5 x 194.8 mm
- board text added: "RJ Buckleup"
- board text added: "ribbon cable"
- board text removed: "designed by Mattia Dal Ben (https://github.com/mattdibi)"
